Commit message: Added new description
Signed-off-by: Juancams <jc.manzanares.serrano@gmail.com>

File: urdf/go2_description.urdf (robot description, URDF)
Before this commit: robot go2_description, 29 links, 28 joints
Links:
- added link camera_link, mass 0
- added link hesai_lidar; collision cylinder length=0.09 radius=0.05; visual cylinder length=0.09 radius=0.05
- added link realsense_link; collision cylinder length=0.09 radius=0.05; visual mesh filename=file://$(find realsense2_description)/meshes/d435.dae
- added link realsense_support_link; collision cylinder length=0.09 radius=0.05; visual cylinder length=0.01 radius=0.01
Joints:
- added joint camera_joint: type fixed, parent Head_upper, child camera_link, origin xyz=0.04 0 0.035 rpy=0 0 0, axis 0 0 0
- added joint hesai_lidar_joint: type fixed, parent base_link, child hesai_lidar, origin xyz=0.15 0 0.12 rpy=0 0 0, axis 0 0 0
- added joint realsense_link_joint: type fixed, parent realsense_support_link, child realsense_link, origin xyz=0.04 0.03 0.018 rpy=0 -0.04 0, axis 0 0 0
- added joint realsense_support_link_joint: type fixed, parent base_link, child realsense_support_link, origin xyz=0.29 0 0.0958 rpy=0 0 0, axis 0 0 0

File: urdf/go2_description.urdf.xacro (robot description, xacro)
@@ -2,5 +2,5 @@
 <robot xmlns:xacro="http://wiki.ros.org/xacro" name="go2">
   <xacro:arg name="prefix" default=""/>
-  <xacro:include filename="$(find go2_description)/urdf/leg.urdf.xacro"/>
+<xacro:include filename="$(find go2_description)/urdf/leg.urdf.xacro"/>
 <!-- Links -->
  <link name="base_link">
@@ -80,4 +80,61 @@
     </inertial>
   </link>
+  <link name="camera_link">
+    <inertial>
+      <origin xyz="0 0 0" rpy="0 0 0" />
+      <mass value="0" />
+      <inertia
+        ixx="0" ixy="0" ixz="0"
+        iyy="0" iyz="0" izz="0" />
+    </inertial>
+  </link>
+  <link name="hesai_lidar">
+    <visual>
+      <origin xyz="0 0 0" rpy="0 0 0" />
+      <geometry>
+        <cylinder radius="0.05" length="0.09" />
+      </geometry>
+      <material name="lidar_color">
+        <color rgba="0.1 0.1 0.1 1" />
+      </material>
+    </visual>
+    <collision>
+      <origin xyz="0 0 0" rpy="0 0 0" />
+      <geometry>
+        <cylinder radius="0.05" length="0.09" />
+      </geometry>
+    </collision>
+  </link>
+  <link name="realsense_support_link">
+    <visual>
+      <origin xyz="0 0 0" rpy="0 0 0" />
+      <geometry>
+        <cylinder radius="0.01" length="0.01" />
+      </geometry>
+      <material name="camera_support_color">
+        <color rgba="0.1 0.1 0.1 1" />
+      </material>
+    </visual>
+    <collision>
+      <origin xyz="0 0 0" rpy="0 0 0" />
+      <geometry>
+        <cylinder radius="0.05" length="0.09" />
+      </geometry>
+    </collision>
+  </link>
+  <link name="realsense_link">
+    <visual>
+      <origin xyz="0 0 0" rpy="1.56 0 1.56" />
+      <geometry>
+        <mesh filename="file://$(find realsense2_description)/meshes/d435.dae" />
+      </geometry>
+    </visual>
+    <collision>
+      <origin xyz="0 0 0" rpy="0 0 0" />
+      <geometry>
+        <cylinder radius="0.05" length="0.09" />
+      </geometry>
+    </collision>
+  </link>
   <joint name="odom_joint" type="fixed">
     <origin xyz="0 0 0" rpy="0 0 0" />
@@ -109,8 +166,31 @@
     <axis xyz="0 0 0" />
   </joint>
-  <xacro:go2_leg name="LF" x_joint="0.1934" y_joint="0.0465" y_thigh_joint="0.0955"/>
-  <xacro:go2_leg name="RF" x_joint="0.1934" y_joint="-0.0465" y_thigh_joint="-0.0955"/>
-  <xacro:go2_leg name="LR" x_joint="-0.1934" y_joint="0.0465" y_thigh_joint="0.0955"/>
+  <joint name="camera_joint" type="fixed">
+    <origin xyz="0.04 0 0.035" rpy="0 0 0" />
+    <parent link="Head_upper" />
+    <child link="camera_link" />
+    <axis xyz="0 0 0" />
+  </joint>
+  <joint name="hesai_lidar_joint" type="fixed">
+    <origin xyz="0.15 0 0.12" rpy="0 0 0" />
+    <parent link="base_link" />
+    <child link="hesai_lidar" />
+    <axis xyz="0 0 0" />
+  </joint>
+  <joint name="realsense_support_link_joint" type="fixed">
+    <origin xyz="0.29 0 0.0958" rpy="0 0 0" />
+    <parent link="base_link" />
+    <child link="realsense_support_link" />
+    <axis xyz="0 0 0" />
+  </joint>
+  <joint name="realsense_link_joint" type="fixed">
+    <origin xyz="0.04 0.03 0.018" rpy="0 -0.04 0" />
+    <parent link="realsense_support_link" />
+    <child link="realsense_link" />
+    <axis xyz="0 0 0" />
+  </joint>
+  <xacro:go2_leg name="FL" x_joint="0.1934" y_joint="0.0465" y_thigh_joint="0.0955"/>
+  <xacro:go2_leg name="FR" x_joint="0.1934" y_joint="-0.0465" y_thigh_joint="-0.0955"/>
+  <xacro:go2_leg name="RL" x_joint="-0.1934" y_joint="0.0465" y_thigh_joint="0.0955"/>
   <xacro:go2_leg name="RR" x_joint="-0.1934" y_joint="-0.0465" y_thigh_joint="-0.0955"/>
-  <xacro:include filename="$(find go2_description)/urdf/gazebo.urdf.xacro"/>
 </robot>

File: urdf/leg.urdf.xacro (robot description, xacro)
@@ -2,18 +2,17 @@
 <robot xmlns:xacro="http://ros.org/wiki/xacro">
   <xacro:macro name="go2_leg" params="name  x_joint y_joint y_thigh_joint" >
-    <!-- <xacro:include filename="$(find go2_description)/urdf/transmission.urdf.xacro"/> -->
-    <xacro:property name="LF" value="LF" />
-    <xacro:property name="RF" value="RF" />
-    <xacro:property name="LR" value="LR" />
+    <xacro:property name="FL" value="FL" />
+    <xacro:property name="FR" value="FR" />
+    <xacro:property name="RL" value="RL" />
     <xacro:property name="RR" value="RR" />
     <link name="${name}_hip">
       <inertial>
-        <xacro:if value="${(name == LF)}">
+        <xacro:if value="${(name == FL)}">
           <origin xyz="-0.0054 0.00194 -0.000105" rpy="0 0 0" />
         </xacro:if>
-        <xacro:if value="${(name == RF)}">
+        <xacro:if value="${(name == FR)}">
           <origin xyz="-0.0054 -0.00194 -0.000105" rpy="0 0 0" />
         </xacro:if>
-        <xacro:if value="${(name == LR)}">
+        <xacro:if value="${(name == RL)}">
           <origin xyz="0.0054 0.00194 -0.000105" rpy="0 0 0" />
         </xacro:if>
@@ -62,10 +61,5 @@
         <origin xyz="0 0 0" rpy="0 0 0" />
         <geometry>
-          <xacro:if value="${(name == LF) or (name == LR)}">
-            <mesh filename="file://$(find go2_description)/dae/thigh.dae" scale="1 1 1"/>
-          </xacro:if>
-           <xacro:if value="${(name == RF) or (name == RR)}">
-            <mesh filename="file://$(find go2_description)/dae/thigh_mirror.dae" scale="1 1 1"/>
-          </xacro:if>
+            <mesh filename="package://go2_description/dae/thigh.dae" />
         </geometry>
         <material
@@ -81,5 +75,5 @@
       </collision>
     </link>
-    <joint name="${name}_upper_leg_joint" type="revolute">
+    <joint name="${name}_upper_leg_joint" type="continuous">
       <origin xyz="0 ${y_thigh_joint} 0" rpy="0 0 0" />
       <parent link="${name}_hip" />
@@ -100,8 +94,8 @@
         <origin xyz="0 0 0" rpy="0 0 0" />
         <geometry>
-          <xacro:if value="${(name == LF) or (name == LR)}">
+          <xacro:if value="${(name == FL) or (name == RL)}">
             <mesh filename="file://$(find go2_description)/dae/calf.dae" scale="1 1 1"/>
           </xacro:if>
-           <xacro:if value="${(name == RF) or (name == RR)}">
+           <xacro:if value="${(name == FR) or (name == RR)}">
             <mesh filename="file://$(find go2_description)/dae/calf_mirror.dae" scale="1 1 1"/>
           </xacro:if>
@@ -157,25 +151,4 @@
       <axis xyz="0 0 0" />
     </joint>
-    <ros2_control name="${name}_control" type="system">
-      <hardware>
-        <plugin>gazebo_ros2_control/GazeboSystem</plugin>
-      </hardware>
-      <joint name="${name}_hip_joint">
-        <command_interface name="effort"/>
-        <state_interface name="position"/>
-        <state_interface name="velocity"/>
-      </joint>
-      <joint name="${name}_upper_leg_joint">
-        <command_interface name="effort"/>
-        <state_interface name="position"/>
-        <state_interface name="velocity"/>
-      </joint>
-      <joint name="${name}_lower_leg_joint">
-        <command_interface name="effort"/>
-        <state_interface name="position"/>
-        <state_interface name="velocity"/>
-      </joint>
-    </ros2_control>
-    <!-- <xacro:leg_transmission name="${name}"/> -->
   </xacro:macro>
 </robot>

Commit message: feat: add front camera to URDF

File: urdf/go2_description.urdf (robot description, URDF)
Before this commit: robot go2_description, 29 links, 28 joints
Links:
- added link front_camera
Joints:
- added joint front_camera_joint: type fixed, parent Head_upper, child front_camera, origin xyz=0.045 0 0.03 rpy=-1.5708 0 -1.5708, axis 0 0 0

File: urdf/go2_description.urdf.xacro (robot description, xacro)
@@ -47,4 +47,11 @@
     </collision>
   </link>
+  <link name="front_camera"/>
+  <joint name="front_camera_joint" type="fixed">
+    <origin xyz="0.045 0 0.03" rpy="-1.5708 0 -1.5708" />
+    <parent link="Head_upper" />
+    <child link="front_camera" />
+    <axis xyz="0 0 0" />
+  </joint>
   <link name="Head_lower">
     <inertial>
