Commit message: URDF was modified. each leg has a macro

File: robots/go2_description.urdf.xacro (robot description, xacro)
@@ -1,36 +1,45 @@
 <?xml version="1.0"?>
-<robot xmlns:xacro="http://wiki.ros.org/xacro" name="go2">
-  <xacro:arg name="prefix" default=""/>
-<xacro:include filename="$(find go2_description)/urdf/leg.urdf.xacro"/>
-<!-- Links -->
- <link name="base_link">
-    <inertial>
-      <origin xyz="0.021112 0 -0.005366" rpy="0 0 0" />
-      <mass value="6.921" />
-      <inertia
-        ixx="0.02448" ixy="0.00012166" ixz="0.0014849"
-        iyy="0.098077" iyz="-3.12E-05" izz="0.107" />
-    </inertial>
-    <visual>
-      <origin xyz="0 0 0" rpy="0 0 0" />
-      <geometry>
-         <mesh filename="file://$(find go2_description)/dae/base.dae" scale="1 1 1"/>
-      </geometry>
-      <material
-        name="">
-        <color rgba="1 1 1 1" />
-      </material>
-    </visual>
-    <collision>
-      <origin rpy="0 0 0" xyz="0 0 0" />
-      <geometry>
-        <box size="0.3762 0.0935 0.114" />
-      </geometry>
-    </collision>
-  </link>
-  <link
+<robot name="go2" xmlns:xacro="http://wiki.ros.org/xacro">
+<!-- Import elements (base + legs) -->
+<xacro:include filename="$(find go2_description)/urdf/base/base.urdf.xacro"/>
+<xacro:include filename="$(find go2_description)/urdf/base/leg.urdf.xacro"/>
+<!-- Global Properties  -->
+<xacro:property name="PI" value="3.1415926535897931"/>
+<!-- Leg Allocations -->
+<xacro:property name="leg_offset_x" value="0.194"/>
+<xacro:property name="leg_offset_y" value="0.0685"/>
+<xacro:property name="leg_offset_z" value="0.0"/>
+<!-- Arguments -->
+<xacro:arg name="prefix" default=""/>
+<xacro:arg name="hesai_lidar" default="false"/>
+<xacro:arg name="livox_lidar" default="false"/>
+<xacro:arg name="realsense" default="false"/>
+<xacro:arg name="name" default="go2"/>
+<!-- Robot elements -->
+<!-- Import sensors -->
+<xacro:include filename="$(find go2_description)/urdf/sensors/hesai.urdf.xacro"/>
+<!-- Robot base -->
+<xacro:go2_base prefix="$(arg prefix)"/>
+<!-- Legs -->
+<xacro:go2_leg prefix="FL_" parent="$(arg prefix)base_link" reflect="false"
+        x="${leg_offset_x}"   y="${leg_offset_y}"   z="${leg_offset_z}"
+        roll="0"      pitch="0"   yaw="0"/>
+<xacro:go2_leg prefix="FR_" parent="$(arg prefix)base_link" reflect="true"
+        x="${leg_offset_x}"   y="-${leg_offset_y}"  z="${leg_offset_z}"
+        roll="${PI}"  pitch="0"   yaw="0"/>
+<xacro:go2_leg prefix="RL_" parent="$(arg prefix)base_link" reflect="false"
+        x="-${leg_offset_x}"  y="${leg_offset_y}"   z="${leg_offset_z}"
+        roll="${PI}"  pitch="0"   yaw="${PI}"/>
+<xacro:go2_leg prefix="RR_" parent="$(arg prefix)base_link" reflect="true"
+        x="-${leg_offset_x}"  y="-${leg_offset_y}"  z="${leg_offset_z}"
+        roll="0"      pitch="0"   yaw="${PI}"/>
+<!-- Sensors -->
+<xacro:hesai_sensor prefix="$(arg prefix)" parent="$(arg prefix)base_link">
+  <origin xyz="0.15 0 0.12" rpy="0 0 ${PI/2}"/>
+</xacro:hesai_sensor>
+  <!-- <link
     name="odom">
-  </link>
-  <link name="Head_upper">
+  </link> -->
+  <!-- <link name="Head_upper">
     <inertial>
       <origin xyz="0 0 0" rpy="0 0 0" />
@@ -46,6 +55,6 @@
       </geometry>
     </collision>
-  </link>
-  <link name="Head_lower">
+  </link> -->
+  <!-- <link name="Head_lower">
     <inertial>
       <origin xyz="0 0 0" rpy="0 0 0" />
@@ -61,6 +70,6 @@
       </geometry>
     </collision>
-  </link>
-  <link name="imu">
+  </link> -->
+  <!-- <link name="imu">
     <inertial>
       <origin xyz="0 0 0" rpy="0 0 0" />
@@ -70,6 +79,6 @@
         iyy="0" iyz="0" izz="0" />
     </inertial>
-  </link>
-  <link name="radar">
+  </link> -->
+  <!-- <link name="radar">
     <inertial>
       <origin xyz="0 0 0" rpy="0 0 0" />
@@ -79,6 +88,6 @@
         iyy="0" iyz="0" izz="0" />
     </inertial>
-  </link>
-  <link name="camera_link">
+  </link> -->
+  <!-- <link name="camera_link">
     <inertial>
       <origin xyz="0 0 0" rpy="0 0 0" />
@@ -88,6 +97,6 @@
         iyy="0" iyz="0" izz="0" />
     </inertial>
-  </link>
-  <link name="hesai_lidar">
+  </link> -->
+  <!-- <link name="hesai_lidar">
     <visual>
       <origin xyz="0 0 0" rpy="0 0 0" />
@@ -105,6 +114,6 @@
       </geometry>
     </collision>
-  </link>
-  <link name="realsense_support_link">
+  </link> -->
+  <!-- <link name="realsense_support_link">
     <visual>
       <origin xyz="0 0 0" rpy="0 0 0" />
@@ -122,6 +131,6 @@
       </geometry>
     </collision>
-  </link>
-  <link name="realsense_link">
+  </link> -->
+  <!-- <link name="realsense_link">
     <visual>
       <origin xyz="0 0 0" rpy="1.56 0 1.56" />
@@ -136,61 +145,61 @@
       </geometry>
     </collision>
-  </link>
-  <joint name="odom_joint" type="fixed">
+  </link> -->
+  <!-- <joint name="odom_joint" type="fixed">
     <origin xyz="0 0 0" rpy="0 0 0" />
     <parent link="odom" />
     <child link="base_link" />
-  </joint>
-  <joint name="Head_upper_joint" type="fixed" dont_collapse="true">
+  </joint> -->
+  <!-- <joint name="Head_upper_joint" type="fixed" dont_collapse="true">
     <origin xyz="0.285 0 0.01" rpy="0 0 0" />
     <parent link="base_link" />
     <child link="Head_upper" />
     <axis xyz="0 0 0" />
-  </joint>
- <joint name="Head_lower_joint" type="fixed" dont_collapse="true">
+  </joint> -->
+ <!-- <joint name="Head_lower_joint" type="fixed" dont_collapse="true">
     <origin xyz="0.008 0 -0.07" rpy="0 0 0" />
     <parent link="Head_upper" />
     <child link="Head_lower" />
     <axis xyz="0 0 0" />
-  </joint>
-  <joint name="imu_joint" type="fixed">
+  </joint> -->
+  <!-- <joint name="imu_joint" type="fixed">
     <origin xyz="-0.02557 0 0.04232" rpy="0 0 0" />
     <parent link="base_link" />
     <child link="imu" />
     <axis xyz="0 0 0" />
-  </joint>
-  <joint name="radar_joint" type="fixed">
+  </joint> -->
+  <!-- <joint name="radar_joint" type="fixed">
     <origin xyz="0.28945 0 -0.046825" rpy="0 2.8782 0" />
     <parent link="base_link" />
     <child link="radar" />
     <axis xyz="0 0 0" />
-  </joint>
-  <joint name="camera_joint" type="fixed">
+  </joint> -->
+  <!-- <joint name="camera_joint" type="fixed">
     <origin xyz="0.04 0 0.035" rpy="0 0 0" />
     <parent link="Head_upper" />
     <child link="camera_link" />
     <axis xyz="0 0 0" />
-  </joint>
-  <joint name="hesai_lidar_joint" type="fixed">
+  </joint> -->
+  <!-- <joint name="hesai_lidar_joint" type="fixed">
     <origin xyz="0.15 0 0.12" rpy="0 0 0" />
     <parent link="base_link" />
     <child link="hesai_lidar" />
     <axis xyz="0 0 0" />
-  </joint>
-  <joint name="realsense_support_link_joint" type="fixed">
+  </joint> -->
+  <!-- <joint name="realsense_support_link_joint" type="fixed">
     <origin xyz="0.29 0 0.0958" rpy="0 0 0" />
     <parent link="base_link" />
     <child link="realsense_support_link" />
     <axis xyz="0 0 0" />
-  </joint>
-  <joint name="realsense_link_joint" type="fixed">
+  </joint> -->
+  <!-- <joint name="realsense_link_joint" type="fixed">
     <origin xyz="0.04 0.03 0.018" rpy="0 -0.04 0" />
     <parent link="realsense_support_link" />
     <child link="realsense_link" />
     <axis xyz="0 0 0" />
-  </joint>
-  <xacro:go2_leg name="FL" x_joint="0.1934" y_joint="0.0465" y_thigh_joint="0.0955"/>
+  </joint> -->
+  <!-- <xacro:go2_leg name="FL" x_joint="0.1934" y_joint="0.0465" y_thigh_joint="0.0955"/>
   <xacro:go2_leg name="FR" x_joint="0.1934" y_joint="-0.0465" y_thigh_joint="-0.0955"/>
   <xacro:go2_leg name="RL" x_joint="-0.1934" y_joint="0.0465" y_thigh_joint="0.0955"/>
-  <xacro:go2_leg name="RR" x_joint="-0.1934" y_joint="-0.0465" y_thigh_joint="-0.0955"/>
+  <xacro:go2_leg name="RR" x_joint="-0.1934" y_joint="-0.0465" y_thigh_joint="-0.0955"/> -->
 </robot>

Commit message: Sensors were added to main URDF file

File: robots/go2_description.urdf.xacro (robot description, xacro)
@@ -8,5 +8,5 @@
 <!-- Leg Allocations -->
 <xacro:property name="leg_offset_x" value="0.194"/>
-<xacro:property name="leg_offset_y" value="0.0685"/>
+<xacro:property name="leg_offset_y" value="0.0465"/>
 <xacro:property name="leg_offset_z" value="0.0"/>
 <!-- Arguments -->
@@ -16,7 +16,25 @@
 <xacro:arg name="realsense" default="false"/>
 <xacro:arg name="name" default="go2"/>
-<!-- Robot elements -->
-<!-- Import sensors -->
+<!-- Sensors -->
+<!-- IMU -->
+<xacro:include filename="$(find go2_description)/urdf/sensors/imu.urdf.xacro"/>
+<xacro:imu_sensor prefix="$(arg prefix)" parent="$(arg prefix)base_link">
+  <origin xyz="-0.02557 0 0.04232" rpy="0 0 0"/>
+</xacro:imu_sensor>
+<!-- camera -->
+<xacro:include filename="$(find go2_description)/urdf/sensors/camera.urdf.xacro"/>
+<xacro:camera_sensor prefix="$(arg prefix)" parent="$(arg prefix)base_link">
+  <origin xyz="0.325 0 0.045" rpy="0 0 0"/>
+</xacro:camera_sensor>
+<!-- radar -->
+<xacro:include filename="$(find go2_description)/urdf/sensors/radar.urdf.xacro"/>
+<xacro:radar_sensor prefix="$(arg prefix)" parent="$(arg prefix)base_link">
+  <origin xyz="0.28945 0 -0.046825" rpy="0 2.8782 0"/>
+</xacro:radar_sensor>
+<!-- hesai lidar -->
 <xacro:include filename="$(find go2_description)/urdf/sensors/hesai.urdf.xacro"/>
+<xacro:hesai_sensor prefix="$(arg prefix)" parent="$(arg prefix)base_link">
+  <origin xyz="0.15 0 0.12" rpy="0 0 ${PI/2}"/>
+</xacro:hesai_sensor>
 <!-- Robot base -->
 <xacro:go2_base prefix="$(arg prefix)"/>
@@ -34,172 +52,3 @@
         x="-${leg_offset_x}"  y="-${leg_offset_y}"  z="${leg_offset_z}"
         roll="0"      pitch="0"   yaw="${PI}"/>
-<!-- Sensors -->
-<xacro:hesai_sensor prefix="$(arg prefix)" parent="$(arg prefix)base_link">
-  <origin xyz="0.15 0 0.12" rpy="0 0 ${PI/2}"/>
-</xacro:hesai_sensor>
-  <!-- <link
-    name="odom">
-  </link> -->
-  <!-- <link name="Head_upper">
-    <inertial>
-      <origin xyz="0 0 0" rpy="0 0 0" />
-      <mass value="0.001" />
-      <inertia
-        ixx="9.6e-06" ixy="0" ixz="0"
-        iyy="9.6e-06" iyz="0" izz="9.6e-06" />
-    </inertial>
-    <collision>
-      <origin xyz="0 0 0" rpy="0 0 0" />
-      <geometry>
-        <cylinder radius="0.05" length="0.09" />
-      </geometry>
-    </collision>
-  </link> -->
-  <!-- <link name="Head_lower">
-    <inertial>
-      <origin xyz="0 0 0" rpy="0 0 0" />
-      <mass value="0.001" />
-      <inertia
-        ixx="9.6e-06" ixy="0" ixz="0"
-        iyy="9.6e-06" iyz="0" izz="9.6e-06" />
-    </inertial>
-    <collision>
-      <origin xyz="0 0 0" rpy="0 0 0" />
-      <geometry>
-        <sphere radius="0.047" />
-      </geometry>
-    </collision>
-  </link> -->
-  <!-- <link name="imu">
-    <inertial>
-      <origin xyz="0 0 0" rpy="0 0 0" />
-      <mass value="0" />
-      <inertia
-        ixx="0" ixy="0" ixz="0"
-        iyy="0" iyz="0" izz="0" />
-    </inertial>
-  </link> -->
-  <!-- <link name="radar">
-    <inertial>
-      <origin xyz="0 0 0" rpy="0 0 0" />
-      <mass value="0" />
-      <inertia
-        ixx="0" ixy="0" ixz="0"
-        iyy="0" iyz="0" izz="0" />
-    </inertial>
-  </link> -->
-  <!-- <link name="camera_link">
-    <inertial>
-      <origin xyz="0 0 0" rpy="0 0 0" />
-      <mass value="0" />
-      <inertia
-        ixx="0" ixy="0" ixz="0"
-        iyy="0" iyz="0" izz="0" />
-    </inertial>
-  </link> -->
-  <!-- <link name="hesai_lidar">
-    <visual>
-      <origin xyz="0 0 0" rpy="0 0 0" />
-      <geometry>
-        <cylinder radius="0.05" length="0.09" />
-      </geometry>
-      <material name="lidar_color">
-        <color rgba="0.1 0.1 0.1 1" />
-      </material>
-    </visual>
-    <collision>
-      <origin xyz="0 0 0" rpy="0 0 0" />
-      <geometry>
-        <cylinder radius="0.05" length="0.09" />
-      </geometry>
-    </collision>
-  </link> -->
-  <!-- <link name="realsense_support_link">
-    <visual>
-      <origin xyz="0 0 0" rpy="0 0 0" />
-      <geometry>
-        <cylinder radius="0.01" length="0.01" />
-      </geometry>
-      <material name="camera_support_color">
-        <color rgba="0.1 0.1 0.1 1" />
-      </material>
-    </visual>
-    <collision>
-      <origin xyz="0 0 0" rpy="0 0 0" />
-      <geometry>
-        <cylinder radius="0.05" length="0.09" />
-      </geometry>
-    </collision>
-  </link> -->
-  <!-- <link name="realsense_link">
-    <visual>
-      <origin xyz="0 0 0" rpy="1.56 0 1.56" />
-      <geometry>
-        <mesh filename="file://$(find realsense2_description)/meshes/d435.dae" />
-      </geometry>
-    </visual>
-    <collision>
-      <origin xyz="0 0 0" rpy="0 0 0" />
-      <geometry>
-        <cylinder radius="0.05" length="0.09" />
-      </geometry>
-    </collision>
-  </link> -->
-  <!-- <joint name="odom_joint" type="fixed">
-    <origin xyz="0 0 0" rpy="0 0 0" />
-    <parent link="odom" />
-    <child link="base_link" />
-  </joint> -->
-  <!-- <joint name="Head_upper_joint" type="fixed" dont_collapse="true">
-    <origin xyz="0.285 0 0.01" rpy="0 0 0" />
-    <parent link="base_link" />
-    <child link="Head_upper" />
-    <axis xyz="0 0 0" />
-  </joint> -->
- <!-- <joint name="Head_lower_joint" type="fixed" dont_collapse="true">
-    <origin xyz="0.008 0 -0.07" rpy="0 0 0" />
-    <parent link="Head_upper" />
-    <child link="Head_lower" />
-    <axis xyz="0 0 0" />
-  </joint> -->
-  <!-- <joint name="imu_joint" type="fixed">
-    <origin xyz="-0.02557 0 0.04232" rpy="0 0 0" />
-    <parent link="base_link" />
-    <child link="imu" />
-    <axis xyz="0 0 0" />
-  </joint> -->
-  <!-- <joint name="radar_joint" type="fixed">
-    <origin xyz="0.28945 0 -0.046825" rpy="0 2.8782 0" />
-    <parent link="base_link" />
-    <child link="radar" />
-    <axis xyz="0 0 0" />
-  </joint> -->
-  <!-- <joint name="camera_joint" type="fixed">
-    <origin xyz="0.04 0 0.035" rpy="0 0 0" />
-    <parent link="Head_upper" />
-    <child link="camera_link" />
-    <axis xyz="0 0 0" />
-  </joint> -->
-  <!-- <joint name="hesai_lidar_joint" type="fixed">
-    <origin xyz="0.15 0 0.12" rpy="0 0 0" />
-    <parent link="base_link" />
-    <child link="hesai_lidar" />
-    <axis xyz="0 0 0" />
-  </joint> -->
-  <!-- <joint name="realsense_support_link_joint" type="fixed">
-    <origin xyz="0.29 0 0.0958" rpy="0 0 0" />
-    <parent link="base_link" />
-    <child link="realsense_support_link" />
-    <axis xyz="0 0 0" />
-  </joint> -->
-  <!-- <joint name="realsense_link_joint" type="fixed">
-    <origin xyz="0.04 0.03 0.018" rpy="0 -0.04 0" />
-    <parent link="realsense_support_link" />
-    <child link="realsense_link" />
-    <axis xyz="0 0 0" />
-  </joint> -->
-  <!-- <xacro:go2_leg name="FL" x_joint="0.1934" y_joint="0.0465" y_thigh_joint="0.0955"/>
-  <xacro:go2_leg name="FR" x_joint="0.1934" y_joint="-0.0465" y_thigh_joint="-0.0955"/>
-  <xacro:go2_leg name="RL" x_joint="-0.1934" y_joint="0.0465" y_thigh_joint="0.0955"/>
-  <xacro:go2_leg name="RR" x_joint="-0.1934" y_joint="-0.0465" y_thigh_joint="-0.0955"/> -->
 </robot>

File: urdf/leg/calf.urdf.xacro (robot description, xacro)
@@ -1,6 +1,10 @@
 <?xml version="1.0"?>
 <robot name="calf" xmlns:xacro="http://www.ros.org/wiki/xacro">
-    <!-- Define a macro for base_link -->
+    <xacro:include filename="$(find go2_description)/urdf/leg/foot.urdf.xacro"/>
+    <!-- Define a macro for calf -->
     <xacro:macro name="go2_calf" params="prefix parent *origin reflect">
+        <xacro:property name="foot_offset_x" value="0.0"/>
+        <xacro:property name="foot_offset_y" value="0.0"/>
+        <xacro:property name="foot_offset_z" value="-0.213"/>
         <joint name="${prefix}calf_joint" type="continuous">
             <parent link="${parent}"/>
@@ -45,4 +49,7 @@
             </collision>
         </link>
+        <xacro:go2_foot prefix="${prefix}" parent="${prefix}calf_link" reflect="${reflect}">
+            <origin xyz="${foot_offset_x} ${foot_offset_y} ${foot_offset_z}" rpy="0 0 0"/>
+        </xacro:go2_foot>
     </xacro:macro>
 </robot>

File: urdf/leg/hip.urdf.xacro (robot description, xacro)
@@ -2,8 +2,8 @@
 <robot name="hip" xmlns:xacro="http://www.ros.org/wiki/xacro">
 <xacro:include filename="$(find go2_description)/urdf/leg/thigh.urdf.xacro"/>
-    <!-- Define a macro for base_link -->
+    <!-- Define a macro for hip -->
     <xacro:macro name="go2_hip" params="prefix parent *origin reflect">
         <xacro:property name="thigh_offset_x" value="0.0"/>
-        <xacro:property name="thigh_offset_y" value="0.09"/>
+        <xacro:property name="thigh_offset_y" value="0.0955"/>
         <xacro:property name="thigh_offset_z" value="0.0"/>
         <xacro:if value="${(prefix == RL_) or (prefix == RR_)}">

File: urdf/leg/thigh.urdf.xacro (robot description, xacro)
@@ -2,9 +2,9 @@
 <robot name="thigh" xmlns:xacro="http://www.ros.org/wiki/xacro">
 <xacro:include filename="$(find go2_description)/urdf/leg/calf.urdf.xacro"/>
-    <!-- Define a macro for base_link -->
+    <!-- Define a macro for thigh -->
     <xacro:macro name="go2_thigh" params="prefix parent *origin reflect">
         <xacro:property name="calf_offset_x" value="0.0"/>
         <xacro:property name="calf_offset_y" value="0.0"/>
-        <xacro:property name="calf_offset_z" value="-0.194"/>
+        <xacro:property name="calf_offset_z" value="-0.213"/>
         <joint name="${prefix}thigh_joint" type="continuous">
             <parent link="${parent}"/>

File: urdf/sensors/hesai.urdf.xacro (robot description, xacro)
@@ -28,4 +28,34 @@
             </inertial>
         </link>
+        <gazebo reference="${prefix}lidar_link">
+            <sensor name='gpu_lidar' type='gpu_lidar'>
+            <pose relative_to="${prefix}lidar_link">0 0 0 0 0 0</pose>
+            <topic>${prefix}lidar_sensor</topic>
+            <update_rate>20</update_rate>
+            <gz_frame_id>${prefix}lidar_link</gz_frame_id>
+            <lidar>
+                <scan>
+                <horizontal>
+                    <samples>450</samples> <!-- 900 -->
+                    <resolution>1</resolution>
+                    <min_angle>-3.141592</min_angle>
+                    <max_angle>3.141592</max_angle>
+                </horizontal>
+                <vertical>
+                    <samples>16</samples>
+                    <resolution>1</resolution>
+                    <min_angle>-0.261799</min_angle>
+                    <max_angle>0.261799</max_angle>
+                </vertical>
+                </scan>
+                <range>
+                <min>0.2</min>
+                <max>90.0</max>
+                <resolution>0.02</resolution>
+                </range>
+            </lidar>
+            <visualize>true</visualize>
+            </sensor>
+        </gazebo>
     </xacro:macro>
 </robot>
